File: test/test.kicad_pcb (KiCad board)
At the start: 2 copper layers, 1 part

Commit message: backup
Parts:
- removed REF**: Arduino_Nano, Module:Arduino_Nano
- added A1: Arduino_Nano_v2.x, Module:Arduino_Nano, F.Cu at (105.8, 75.8)
- added C2: 100h, Capacitor_THT:C_Disc_D3.0mm_W1.6mm_P2.50mm, F.Cu at (210.0, 42.8)
- added C3: C, Capacitor_THT:C_Disc_D3.0mm_W1.6mm_P2.50mm, F.Cu at (210.0, 46.9)
- added C4: 100h, Capacitor_THT:C_Disc_D3.0mm_W1.6mm_P2.50mm, F.Cu at (210.0, 51.1)
- added C5: 100h, Capacitor_THT:C_Disc_D3.0mm_W1.6mm_P2.50mm, F.Cu at (210.0, 55.2)
- added C6: C, Capacitor_THT:C_Disc_D3.0mm_W1.6mm_P2.50mm, F.Cu at (210.0, 59.4)
- added C7: 100h, Capacitor_THT:C_Disc_D3.0mm_W1.6mm_P2.50mm, F.Cu at (210.0, 63.5)
- added D1: D, Diode_THT:D_5W_P5.08mm_Vertical_AnodeUp, F.Cu at (223.9, 45.5)
- added D2: D, Diode_THT:D_5W_P5.08mm_Vertical_AnodeUp, F.Cu at (223.9, 55.0)
- added D3: LED, LED_THT:LED_D3.0mm, F.Cu at (236.1, 43.0)
- added D4: LED, LED_THT:LED_D3.0mm, F.Cu at (236.1, 52.3)
- added R1: 10K, Resistor_THT:R_Axial_DIN0204_L3.6mm_D1.6mm_P1.90mm_Vertical, F.Cu at (183.1, 41.7)
- added R10: 10K, Resistor_THT:R_Axial_DIN0204_L3.6mm_D1.6mm_P1.90mm_Vertical, F.Cu at (188.1, 48.0)
- added R11: 10K, Resistor_THT:R_Axial_DIN0204_L3.6mm_D1.6mm_P1.90mm_Vertical, F.Cu at (188.1, 51.1)
- added R12: 1K, Resistor_THT:R_Axial_DIN0204_L3.6mm_D1.6mm_P1.90mm_Vertical, F.Cu at (188.1, 54.3)
- added R13: 10K, Resistor_THT:R_Axial_DIN0204_L3.6mm_D1.6mm_P1.90mm_Vertical, F.Cu at (188.1, 57.5)
- added R14: 10K, Resistor_THT:R_Axial_DIN0204_L3.6mm_D1.6mm_P1.90mm_Vertical, F.Cu at (193.1, 41.7)
- added R15: 510K, Resistor_THT:R_Axial_DIN0204_L3.6mm_D1.6mm_P1.90mm_Vertical, F.Cu at (193.1, 44.9)
- added R16: 1K, Resistor_THT:R_Axial_DIN0204_L3.6mm_D1.6mm_P1.90mm_Vertical, F.Cu at (193.1, 48.0)
- added R17: 10K, Resistor_THT:R_Axial_DIN0204_L3.6mm_D1.6mm_P1.90mm_Vertical, F.Cu at (193.1, 51.1)
- added R18: 1K, Resistor_THT:R_Axial_DIN0204_L3.6mm_D1.6mm_P1.90mm_Vertical, F.Cu at (193.1, 54.3)
- added R2: 1K, Resistor_THT:R_Axial_DIN0204_L3.6mm_D1.6mm_P1.90mm_Vertical, F.Cu at (183.1, 44.9)
- added R3: 1K, Resistor_THT:R_Axial_DIN0204_L3.6mm_D1.6mm_P1.90mm_Vertical, F.Cu at (73.0, 56.5)
- added R5: 10K, Resistor_THT:R_Axial_DIN0204_L3.6mm_D1.6mm_P1.90mm_Vertical, F.Cu at (183.1, 51.1)
- added R6: 4.7K, Resistor_THT:R_Axial_DIN0204_L3.6mm_D1.6mm_P1.90mm_Vertical, F.Cu at (183.1, 54.3)
- added R7: 4.7K, Resistor_THT:R_Axial_DIN0204_L3.6mm_D1.6mm_P1.90mm_Vertical, F.Cu at (183.1, 57.5)
- added R8: 1K, Resistor_THT:R_Axial_DIN0204_L3.6mm_D1.6mm_P1.90mm_Vertical, F.Cu at (188.1, 41.7)
- added R9: 510K, Resistor_THT:R_Axial_DIN0204_L3.6mm_D1.6mm_P1.90mm_Vertical, F.Cu at (188.1, 44.9)
- added SW2: SW_Push, Button_Switch_THT:SW_PUSH_6mm, F.Cu at (163.3, 74.0)
- added U2: ~, my_lib:dfplayer_mini, F.Cu at (122.0, 52.0)
- added U3: ~, my_lib:cd40106be, F.Cu at (142.0, 112.0)

Commit message: backup
Parts:
- added J1: Conn_01x02_Pin, Connector_PinHeader_1.00mm:PinHeader_1x02_P1.00mm_Horizontal, F.Cu at (133.6, 87.5)
- added J2: Conn_01x02_Pin, Connector_PinHeader_1.00mm:PinHeader_1x02_P1.00mm_Horizontal, F.Cu at (133.6, 90.5)
- moved R2 93.1 mm to (102.0, 90.5)
- moved R3 42.1 mm to (102.0, 87.0)
- moved SW2 16.3 mm to (147.0, 73.0)
- moved A1 12.3 mm to (107.9, 88.0)
- moved U3 8.51 mm to (150.5, 112.5)
