File: test/test.kicad_sch (KiCad schematic)
At the start: 33 parts, among them SW2 SW_Push, SW3 SW_Push, SW4 SW_Push

Commit message: backup
Parts:
- removed SW3, SW4: SW_Push, symbol Switch:SW_Push
- added SW1, SW3: SW_SPST, symbol Switch:SW_SPST
- C2, C3, C4, C5, C6, C7: footprint (none) -> Capacitor_THT:C_Disc_D3.0mm_W1.6mm_P2.50mm
- D1, D2: footprint (none) -> Diode_THT:D_5W_P5.08mm_Vertical_AnodeUp
- D3, D4: footprint (none) -> LED_THT:LED_D3.0mm
- R1, R10, R11, R12, R13, R14, R15, R16, R17, R18, R2, R3, R5, R6, R7, R8, R9: footprint (none) -> Resistor_THT:R_Axial_DIN0204_L3.6mm_D1.6mm_P1.90mm_Vertical
- SW2: footprint (none) -> Button_Switch_THT:SW_PUSH_6mm
- U2: footprint (none) -> my_lib:dfplayer_mini
- U3: footprint (none) -> my_lib:cd40106be
Connections:
- net A: now also SW1.1 (A)
- net C: now also SW3.1 (A)
- net GND: now also SW1.2 (B), SW3.2 (B)
Other:
- note added: "Master Button"
- note removed: "Buttons"

Commit message: backup
Parts:
- removed SW1, SW3: SW_SPST, symbol Switch:SW_SPST
- added J1, J2: Conn_01x02_Pin, Connector_PinHeader_1.00mm:PinHeader_1x02_P1.00mm_Horizontal, symbol Connector:Conn_01x02_Pin
Connections:
- net A: now also J1.1 (Pin_1)
- net C: now also J2.1 (Pin_1)
- net GND: now also J1.2 (Pin_2), J2.2 (Pin_2)
- no-connect marks 0 -> 33
